File: CAN_commodo.kicad_sch (KiCad schematic)
At the start: 0 parts

Commit message: added buck
Parts:
- added C27: 10uF, Capacitor_SMD:C_0402_1005Metric, symbol Device:C
- added C36: 100nF, Capacitor_SMD:C_0402_1005Metric, symbol Device:C
- added C39: 100pF, Capacitor_SMD:C_0402_1005Metric, symbol Device:C
- added L2: 3.3uH, sthymuli:FXL0630-3R3-M, symbol Device:L
- added R38: 47K, Capacitor_SMD:C_0201_0603Metric, symbol Device:R
- added R39: 15K, Capacitor_SMD:C_0201_0603Metric, symbol Device:R
- added U1: ESP32-C3_SUPERMINI_TH, ESP32-C3_SUPERMINI_TH:MODULE_ESP32-C3_SUPERMINI_TH, symbol ESP32-C3_SUPERMINI_TH:ESP32-C3_SUPERMINI_TH
- added U4: AP62300WU, Package_TO_SOT_SMD:TSOT-23-6, symbol Regulator_Switching:AP62300WU
Connections:
- new net: C39.1, R38.2, R39.1, U4.4 (FB)
- new net: C39.2, L2.2, R38.1
- new net: C27.1, U4.3 (IN)
- new net: C36.1, U4.6 (BST)
- new net: C36.2, L2.1, U4.2 (SW)
- new net GND: C27.2, R39.2, U4.1 (GND)
- no-connect marks 0 -> 1
Other:
- note added: "150 uA quiescent"
- note added: "3V3 rail"
- note added: "DC buck, IOUT=3A"
- note added: "Leave floating for automatic startup"
